Commit message: add 3dofs to the connection joint

File: custom_description/urdf/connected_robots/connected_robot.xacro (robot description, xacro)
@@ -1,43 +1,40 @@
 <?xml version="1.0"?>
 <robot xmlns:xacro="http://www.ros.org/wiki/xacro" name="connected_robot">
-    <xacro:arg name="sim" default="false"/>
-    <xacro:include filename="$(find custom_description)/urdf/connected_robots/robot_macro.xacro"/>
+    <xacro:arg name="sim" default="false" />
+    <xacro:include filename="$(find custom_description)/urdf/connected_robots/robot_macro.xacro" />
+    <xacro:include filename="$(find custom_description)/urdf/connected_robots/spherical_joint.xacro" />
     <link name="rod">
         <visual>
-            <origin rpy="0 0 0" xyz="0 0 0"/>
+            <origin rpy="${pi/2} 0 0" xyz="0 0 0" />
             <geometry>
-                <box size="0.1 1 0.1"/>
+                <cylinder length="1" radius="0.03" />
             </geometry>
         </visual>
-        <collision>
-            <origin rpy="0 0 0" xyz="0 0 0"/>
+        <!-- <collision>
+            <origin rpy="0 0 0" xyz="0 0 0" />
             <geometry>
-                <box size="0.1 1 0.1"/>
+                <cylinder length="1" radius="0.1" />
             </geometry>
-        </collision>
-        <!-- <inertial>
-            <origin rpy="0 0 0" xyz="$0 0 0"/>
-            <mass value="1"/>
+        </collision> -->
+        <inertial>
+            <origin rpy="0 0 0" xyz="0 0 0" />
+            <mass value="0.1" />
             <inertia
-                    ixx="0.1" ixy="0.01" ixz="0.01"
-                    iyy="0.1" iyz="0.01"
-                    izz="0.1"/>
-        </inertial> -->
+                ixx="0.1" ixy="0.01" ixz="0.01"
+                iyy="0.1" iyz="0.01"
+                izz="0.1" />
+        </inertial>
     </link>
-    <xacro:legged_robot robot_type="aliengo" ns="alien1" prefix="alien1_" sim="$(arg sim)" >
-        <origin rpy="0 0 0" xyz="0 -0.5 -0.1"/>
+    <xacro:ball_joint name="alien1_ball" parent="rod" child="alien1_base">
+        <origin rpy="0 0 0" xyz="0 -0.5 0" />
+    </xacro:ball_joint>
+    <xacro:legged_robot robot_type="aliengo" ns="alien1" prefix="alien1_" sim="$(arg sim)">
+        <origin rpy="0 0 0" xyz="0 -0.5 -0.1" />
     </xacro:legged_robot>
-    <joint name="alien1_rod_joint" type="fixed">
-        <origin rpy="0 0 0" xyz="0 -0.5 -0.1"/>
-        <parent link="rod" />
-        <child link="alien1_base" />
-    </joint>
-    <xacro:legged_robot robot_type="aliengo" ns="alien2" prefix="alien2_" sim="$(arg sim)" >
-        <origin rpy="0 0 0" xyz="0 0.5 -0.1"/>
+    <xacro:ball_joint name="alien2_ball" parent="rod" child="alien2_base">
+        <origin rpy="0 0 0" xyz="0 0.5 0" />
+    </xacro:ball_joint>
+    <xacro:legged_robot robot_type="aliengo" ns="alien2" prefix="alien2_" sim="$(arg sim)">
+        <origin rpy="0 0 0" xyz="0 0.5 -0.1" />
     </xacro:legged_robot>
-    <joint name="alien2_rod_joint" type="fixed">
-        <origin rpy="0 0 0" xyz="0 0.5 -0.1"/>
-        <parent link="rod" />
-        <child link="alien2_base" />
-    </joint>
 </robot>

File: custom_description/urdf/connected_robots/robot_macro.xacro (robot description, xacro)
@@ -11,10 +11,4 @@
             value="package://legged_unitree_description/meshes/${robot_type}" />
         <link name="${prefix}base">
-            <visual>
-                <xacro:insert_block name="origin"/>
-            </visual>
-            <collision>
-                <xacro:insert_block name="origin"/>
-            </collision>
         </link>
         <joint name="${prefix}trunk_joint" type="fixed">

File: custom_description/urdf/sensor_t265.xacro (robot description, xacro)
@@ -30,14 +30,14 @@
             <visual>
                 <origin xyz="0 0 0" rpy="0 0 0"/>
-                <geometry>
-                    <!-- <mesh filename="package://realsense2_description/meshes/t265.stl"/> -->
-                </geometry>
+                <!-- <geometry>
+                    <mesh filename="package://realsense2_description/meshes/t265.stl"/>
+                </geometry> -->
                 <material name="${name}_aluminum"/>
             </visual>
             <collision>
                 <origin xyz="0 0 0" rpy="0 0 0"/>
-                <geometry>
-                    <!-- <mesh filename="package://realsense2_description/meshes/t265.stl"/> -->
-                </geometry>
+                <!-- <geometry>
+                    <mesh filename="package://realsense2_description/meshes/t265.stl"/>
+                </geometry> -->
             </collision>
             <inertial>

Commit message: update on worlds and xacro files

File: custom_description/urdf/connected_robots/connected_robot.xacro (robot description, xacro)
@@ -2,39 +2,15 @@
 <robot xmlns:xacro="http://www.ros.org/wiki/xacro" name="connected_robot">
     <xacro:arg name="sim" default="false" />
+    <xacro:arg name="robot_type" default="aliengo" />
+    <xacro:arg name="ns_1" default="" />
+    <xacro:arg name="ns_2" default="" />
     <xacro:include filename="$(find custom_description)/urdf/connected_robots/robot_macro.xacro" />
-    <xacro:include filename="$(find custom_description)/urdf/connected_robots/spherical_joint.xacro" />
-    <link name="rod">
-        <visual>
-            <origin rpy="${pi/2} 0 0" xyz="0 0 0" />
-            <geometry>
-                <cylinder length="1" radius="0.03" />
-            </geometry>
-        </visual>
-        <!-- <collision>
-            <origin rpy="0 0 0" xyz="0 0 0" />
-            <geometry>
-                <cylinder length="1" radius="0.1" />
-            </geometry>
-        </collision> -->
-        <inertial>
-            <origin rpy="0 0 0" xyz="0 0 0" />
-            <mass value="0.1" />
-            <inertia
-                ixx="0.1" ixy="0.01" ixz="0.01"
-                iyy="0.1" iyz="0.01"
-                izz="0.1" />
-        </inertial>
-    </link>
-    <xacro:ball_joint name="alien1_ball" parent="rod" child="alien1_base">
-        <origin rpy="0 0 0" xyz="0 -0.5 0" />
-    </xacro:ball_joint>
-    <xacro:legged_robot robot_type="aliengo" ns="alien1" prefix="alien1_" sim="$(arg sim)">
+    <xacro:include filename="$(find custom_description)/urdf/connected_robots/rod_with_joints_macro.xacro" />
+    <xacro:legged_robot robot_type="$(arg robot_type)" ns="$(arg ns_1)" prefix="$(arg ns_1)_" sim="$(arg sim)">
         <origin rpy="0 0 0" xyz="0 -0.5 -0.1" />
     </xacro:legged_robot>
-    <xacro:ball_joint name="alien2_ball" parent="rod" child="alien2_base">
-        <origin rpy="0 0 0" xyz="0 0.5 0" />
-    </xacro:ball_joint>
-    <xacro:legged_robot robot_type="aliengo" ns="alien2" prefix="alien2_" sim="$(arg sim)">
+    <xacro:legged_robot robot_type="$(arg robot_type)" ns="$(arg ns_2)" prefix="$(arg ns_2)_" sim="$(arg sim)">
         <origin rpy="0 0 0" xyz="0 0.5 -0.1" />
     </xacro:legged_robot>
+    <xacro:rod_with_joints first_robot="$(arg ns_1)" second_robot="$(arg ns_2)" />
 </robot>
