Commit message: edit package names

File: custom_description/urdf/robot.xacro (robot description, xacro)
@@ -8,6 +8,6 @@
     <xacro:include filename="$(find legged_unitree_description)/urdf/common/imu.xacro"/>
     <xacro:include filename="$(find legged_unitree_description)/urdf/$(arg robot_type)/const.xacro"/>
-    <xacro:include filename="$(find fieldai_legged_perceptive_description)/urdf/sensor_d435.xacro"/>
-    <xacro:include filename="$(find fieldai_legged_perceptive_description)/urdf/sensor_t265.xacro"/>
+    <xacro:include filename="$(find custom_description)/urdf/sensor_d435.xacro"/>
+    <xacro:include filename="$(find custom_description)/urdf/sensor_t265.xacro"/>
     <xacro:property name="mesh_path" value="package://legged_unitree_description/meshes/$(arg robot_type)"/>
     <link name="base">
@@ -63,5 +63,5 @@
             <origin rpy="0 0 0" xyz="0 0 0"/>
             <geometry>
-                <!-- <mesh filename="package://fieldai_legged_perceptive_description/meshes/$(arg robot_type)/aliengo_payload.dae" scale="1 1 1"/> -->
+                <!-- <mesh filename="package://custom_description/meshes/$(arg robot_type)/aliengo_payload.dae" scale="1 1 1"/> -->
                 <box size="0.2 0.2 0.2"/>
             </geometry>

File: custom_description/urdf/sensor_d435.xacro (robot description, xacro)
@@ -112,5 +112,5 @@
             </joint>
             <link name="${name}_color_optical_frame"/>
-            <xacro:include filename="$(find fieldai_legged_perceptive_description)/urdf/gazebo_d435.xacro"/>
+            <xacro:include filename="$(find custom_description)/urdf/gazebo_d435.xacro"/>
             <!-- Realsense Gazebo Plugin -->
     <xacro:gazebo_d435 camera_name="${name}" reference_link="${name}_link" topics_ns="${topics_ns}" depth_optical_frame="${name}_depth_optical_frame" color_optical_frame="${name}_color_optical_frame" infrared1_optical_frame="${name}_left_ir_optical_frame" infrared2_optical_frame="${name}_right_ir_optical_frame"/>

Commit message: Modified LeggedHWSim

File: custom_description/urdf/robot.xacro (robot description, xacro)
@@ -3,7 +3,7 @@
     <xacro:arg name="sim" default="false"/>
     <xacro:arg name="robot_type" default="a1"/>
+    <xacro:arg name="ns" default=""/>
     <xacro:include filename="$(find legged_unitree_description)/urdf/common/materials.xacro"/>
     <xacro:include filename="$(find legged_unitree_description)/urdf/common/leg.xacro"/>
-    <xacro:include filename="$(find legged_unitree_description)/urdf/common/gazebo.xacro"/>
     <xacro:include filename="$(find legged_unitree_description)/urdf/common/imu.xacro"/>
     <xacro:include filename="$(find legged_unitree_description)/urdf/$(arg robot_type)/const.xacro"/>
@@ -63,17 +63,30 @@
             <origin rpy="0 0 0" xyz="0 0 0"/>
             <geometry>
-                <!-- <mesh filename="package://custom_description/meshes/$(arg robot_type)/aliengo_payload.dae" scale="1 1 1"/> -->
-                <box size="0.2 0.2 0.2"/>
+                <mesh filename="package://custom_description/meshes/$(arg robot_type)/aliengo_payload.dae" scale="1 1 1"/>
             </geometry>
         </visual>
-        <!-- <collision>
-               <origin rpy="0 0 0" xyz="0 0 0"/>
-                <geometry>
-                    <mesh filename="package://aliengo_description/meshes/aliengo_payload.dae" scale="1 1 1"/>
-                </geometry>
-        </collision> -->
     </link>
     <xacro:sensor_d435 name="front_camera" topics_ns="front_camera" parent="base">
            <origin xyz="0.16 0.048 0.30" rpy="0 0.54359877559 0"/>
     </xacro:sensor_d435>
+    <!-- ros_control plugin -->
+    <gazebo>
+        <plugin name="gazebo_ros_control" filename="libcustom_legged_hw_sim.so">
+            <robotNamespace>/$(arg ns)</robotNamespace>
+            <robotParam>legged_robot_description</robotParam>
+            <robotSimType>custom_gazebo/CustomLeggedHWSim</robotSimType>
+        </plugin>
+    </gazebo>
+    <gazebo>
+        <plugin name="p3d_base_controller" filename="libgazebo_ros_p3d.so">
+            <alwaysOn>true</alwaysOn>
+            <updateRate>1000.0</updateRate>
+            <bodyName>base</bodyName>
+            <topicName>ground_truth/state</topicName>
+            <gaussianNoise>0</gaussianNoise>
+            <frameName>world</frameName>
+            <xyzOffsets>0 0 0</xyzOffsets>
+            <rpyOffsets>0 0 0</rpyOffsets>
+        </plugin>
+    </gazebo>
 </robot>

Commit message: remove the payload

File: custom_description/urdf/robot.xacro (robot description, xacro)
@@ -49,5 +49,5 @@
          <origin xyz="0.35 0.0 0.0" rpy="0.0 -0.05 -0.0"/>
     </xacro:sensor_t265>
-    <joint name="payload_joint" type="fixed">
+    <!-- <joint name="payload_joint" type="fixed">
         <parent link="base" />
         <child link="payload" />
@@ -65,5 +65,5 @@
             </geometry>
         </visual>
-    </link>
+    </link> -->
     <xacro:sensor_d435 name="front_camera" topics_ns="$(arg ns)/front_camera" parent="base">
            <origin xyz="0.16 0.048 0.30" rpy="0 0.54359877559 0"/>

Commit message: add hardware setup

File: custom_description/urdf/robot.xacro (robot description, xacro)
@@ -1,51 +1,56 @@
 <?xml version="1.0"?>
 <robot xmlns:xacro="http://www.ros.org/wiki/xacro" name="robot">
-    <xacro:arg name="sim" default="false"/>
-    <xacro:arg name="robot_type" default="a1"/>
-    <xacro:arg name="ns" default=""/>
-    <xacro:include filename="$(find legged_unitree_description)/urdf/common/materials.xacro"/>
-    <xacro:include filename="$(find legged_unitree_description)/urdf/common/leg.xacro"/>
-    <xacro:include filename="$(find legged_unitree_description)/urdf/common/imu.xacro"/>
-    <xacro:include filename="$(find legged_unitree_description)/urdf/$(arg robot_type)/const.xacro"/>
-    <xacro:include filename="$(find custom_description)/urdf/sensor_d435.xacro"/>
-    <xacro:include filename="$(find custom_description)/urdf/sensor_t265.xacro"/>
-    <xacro:property name="mesh_path" value="package://legged_unitree_description/meshes/$(arg robot_type)"/>
+    <xacro:arg name="sim" default="false" />
+    <xacro:arg name="robot_type" default="a1" />
+    <xacro:arg name="ns" default="" />
+    <xacro:include filename="$(find legged_unitree_description)/urdf/common/materials.xacro" />
+    <xacro:include filename="$(find legged_unitree_description)/urdf/common/leg.xacro" />
+    <xacro:include filename="$(find legged_unitree_description)/urdf/common/imu.xacro" />
+    <xacro:include filename="$(find legged_unitree_description)/urdf/$(arg robot_type)/const.xacro" />
+    <xacro:include filename="$(find custom_description)/urdf/sensor_d435.xacro" />
+    <xacro:include filename="$(find custom_description)/urdf/sensor_t265.xacro" />
+    <xacro:property name="mesh_path"
+        value="package://legged_unitree_description/meshes/$(arg robot_type)" />
     <link name="base">
         <visual>
-            <origin rpy="0 0 0" xyz="0 0 0"/>
+            <origin rpy="0 0 0" xyz="0 0 0" />
             <geometry>
-                <mesh filename="${mesh_path}/trunk.dae" scale="1 1 1"/>
+                <mesh filename="${mesh_path}/trunk.dae" scale="1 1 1" />
             </geometry>
         </visual>
         <collision>
-            <origin rpy="0 0 0" xyz="0 0 0"/>
+            <origin rpy="0 0 0" xyz="0 0 0" />
             <geometry>
-                <box size="${trunk_length} ${trunk_width} ${trunk_height}"/>
+                <box size="${trunk_length} ${trunk_width} ${trunk_height}" />
             </geometry>
         </collision>
         <inertial>
-            <origin rpy="0 0 0" xyz="${trunk_com_x} ${trunk_com_y} ${trunk_com_z}"/>
-            <mass value="${trunk_mass}"/>
+            <origin rpy="0 0 0" xyz="${trunk_com_x} ${trunk_com_y} ${trunk_com_z}" />
+            <mass value="${trunk_mass}" />
             <inertia
-                    ixx="${trunk_ixx}" ixy="${trunk_ixy}" ixz="${trunk_ixz}"
-                    iyy="${trunk_iyy}" iyz="${trunk_iyz}"
-                    izz="${trunk_izz}"/>
+                ixx="${trunk_ixx}" ixy="${trunk_ixy}" ixz="${trunk_ixz}"
+                iyy="${trunk_iyy}" iyz="${trunk_iyz}"
+                izz="${trunk_izz}" />
         </inertial>
     </link>
-    <xacro:IMU connected_to="base" imu_name="base_imu" xyz="0. 0. 0." rpy="0. 0. 0."/>
-    <xacro:leg prefix="LF" mesh_path="${mesh_path}" mirror="1" mirror_dae="True" front_hind="1" front_hind_dae="True">
-        <origin rpy="0 0 0" xyz="${leg_offset_x} ${leg_offset_y} 0"/>
+    <xacro:IMU connected_to="base" imu_name="base_imu" xyz="0. 0. 0." rpy="0. 0. 0." />
+    <xacro:leg prefix="LF" mesh_path="${mesh_path}" mirror="1" mirror_dae="True" front_hind="1"
+        front_hind_dae="True">
+        <origin rpy="0 0 0" xyz="${leg_offset_x} ${leg_offset_y} 0" />
     </xacro:leg>
-    <xacro:leg prefix="LH" mesh_path="${mesh_path}" mirror="1" mirror_dae="True" front_hind="-1" front_hind_dae="False">
-        <origin rpy="0 0 0" xyz="${-leg_offset_x} ${leg_offset_y} 0"/>
+    <xacro:leg prefix="LH" mesh_path="${mesh_path}" mirror="1" mirror_dae="True" front_hind="-1"
+        front_hind_dae="False">
+        <origin rpy="0 0 0" xyz="${-leg_offset_x} ${leg_offset_y} 0" />
     </xacro:leg>
-    <xacro:leg prefix="RF" mesh_path="${mesh_path}" mirror="-1" mirror_dae="False" front_hind="1" front_hind_dae="True">
-        <origin rpy="0 0 0" xyz="${leg_offset_x} ${-leg_offset_y} 0"/>
+    <xacro:leg prefix="RF" mesh_path="${mesh_path}" mirror="-1" mirror_dae="False" front_hind="1"
+        front_hind_dae="True">
+        <origin rpy="0 0 0" xyz="${leg_offset_x} ${-leg_offset_y} 0" />
     </xacro:leg>
-    <xacro:leg prefix="RH" mesh_path="${mesh_path}" mirror="-1" mirror_dae="False" front_hind="-1" front_hind_dae="False">
-        <origin rpy="0 0 0" xyz="${-leg_offset_x} ${-leg_offset_y} 0"/>
+    <xacro:leg prefix="RH" mesh_path="${mesh_path}" mirror="-1" mirror_dae="False" front_hind="-1"
+        front_hind_dae="False">
+        <origin rpy="0 0 0" xyz="${-leg_offset_x} ${-leg_offset_y} 0" />
     </xacro:leg>
     <xacro:sensor_t265 name="tracking_camera" topics_ns="$(arg ns)/tracking_camera" parent="base">
-         <origin xyz="0.35 0.0 0.0" rpy="0.0 -0.05 -0.0"/>
+        <origin xyz="0.35 0.0 0.0" rpy="0.0 -0.05 -0.0" />
     </xacro:sensor_t265>
     <!-- <joint name="payload_joint" type="fixed">
@@ -66,26 +71,29 @@
         </visual>
     </link> -->
-    <xacro:sensor_d435 name="front_camera" topics_ns="$(arg ns)/front_camera" parent="base">
-           <origin xyz="0.16 0.048 0.30" rpy="0 0.54359877559 0"/>
+    <xacro:sensor_d435 name="front_camera" topics_ns="$(arg ns)/front_camera" parent="base"
+        sim="$(arg sim)">
+        <origin xyz="0.16 0.048 0.30" rpy="0 0.54359877559 0" />
     </xacro:sensor_d435>
     <!-- ros_control plugin -->
-    <gazebo>
-        <plugin name="gazebo_ros_control" filename="libcustom_legged_hw_sim.so">
-            <robotNamespace>/$(arg ns)</robotNamespace>
-            <robotParam>legged_robot_description</robotParam>
-            <robotSimType>custom_gazebo/CustomLeggedHWSim</robotSimType>
-        </plugin>
-    </gazebo>
-    <gazebo>
-        <plugin name="p3d_base_controller" filename="libgazebo_ros_p3d.so">
-            <alwaysOn>true</alwaysOn>
-            <updateRate>1000.0</updateRate>
-            <bodyName>base</bodyName>
-            <topicName>ground_truth/state</topicName>
-            <gaussianNoise>0</gaussianNoise>
-            <frameName>world</frameName>
-            <xyzOffsets>0 0 0</xyzOffsets>
-            <rpyOffsets>0 0 0</rpyOffsets>
-        </plugin>
-    </gazebo>
+    <xacro:if value="$(arg sim)">
+        <gazebo>
+            <plugin name="gazebo_ros_control" filename="libcustom_legged_hw_sim.so">
+                <robotNamespace>/$(arg ns)</robotNamespace>
+                <robotParam>legged_robot_description</robotParam>
+                <robotSimType>custom_gazebo/CustomLeggedHWSim</robotSimType>
+            </plugin>
+        </gazebo>
+        <gazebo>
+            <plugin name="p3d_base_controller" filename="libgazebo_ros_p3d.so">
+                <alwaysOn>true</alwaysOn>
+                <updateRate>1000.0</updateRate>
+                <bodyName>base</bodyName>
+                <topicName>ground_truth/state</topicName>
+                <gaussianNoise>0</gaussianNoise>
+                <frameName>world</frameName>
+                <xyzOffsets>0 0 0</xyzOffsets>
+                <rpyOffsets>0 0 0</rpyOffsets>
+            </plugin>
+        </gazebo>
+    </xacro:if>
 </robot>

Commit message: change the camera pose

File: custom_description/urdf/robot.xacro (robot description, xacro)
@@ -73,5 +73,5 @@
     <xacro:sensor_d435 name="front_camera" topics_ns="$(arg ns)/front_camera" parent="base"
         sim="$(arg sim)">
-        <origin xyz="0.16 0.048 0.30" rpy="0 0.54359877559 0" />
+        <origin xyz="0.22 0.0 0.05" rpy="0 0.21 0" />
     </xacro:sensor_d435>
     <!-- ros_control plugin -->

Commit message: add some config

File: custom_description/urdf/robot.xacro (robot description, xacro)
@@ -52,5 +52,6 @@
     </xacro:leg>
     <xacro:sensor_t265 name="tracking_camera" topics_ns="$(arg ns)/tracking_camera" parent="base">
-        <origin xyz="0.35 0.0 0.0" rpy="0.0 -0.05 -0.0" />
+        <!-- <origin xyz="-0.1 0.0 0.07" rpy="0.0 0.0 -0.0" /> -->
+        <origin xyz="0.22 0.0 0.05" rpy="0 0.21 0" />
     </xacro:sensor_t265>
     <!-- <joint name="payload_joint" type="fixed">

File: custom_description/urdf/sensor_t265.xacro (robot description, xacro)
@@ -30,7 +30,9 @@
             <visual>
                 <origin xyz="0 0 0" rpy="0 0 0"/>
-                <!-- <geometry>
-                    <mesh filename="package://realsense2_description/meshes/t265.stl"/>
-                </geometry> -->
+                <geometry>
+                    <mesh
+                    filename="package://realsense2_description/meshes/t265_full.stl"
+                    scale="0.001 0.001 0.001"/>
+                </geometry>
                 <material name="${name}_aluminum"/>
             </visual>

Commit message: add correct camera location

File: custom_description/urdf/robot.xacro (robot description, xacro)
@@ -53,20 +53,21 @@
     <xacro:sensor_t265 name="tracking_camera" topics_ns="$(arg ns)/tracking_camera" parent="base">
         <!-- <origin xyz="-0.1 0.0 0.07" rpy="0.0 0.0 -0.0" /> -->
-        <origin xyz="0.22 0.0 0.05" rpy="0 0.21 0" />
+        <origin xyz="0.17 0.0 0.07" rpy="0 0.0 0" />
     </xacro:sensor_t265>
     <!-- <joint name="payload_joint" type="fixed">
         <parent link="base" />
         <child link="payload" />
-        <origin rpy="0 0 0" xyz="0 0 0.13" />
+        <origin rpy="0.0 0.0 0.0" xyz="0.21 0 0.07" />
     </joint>
     <link name="payload">
         <inertial>
-            <mass value="3" />
+            <mass value="0.03" />
             <origin rpy="0 0 0" xyz="0 0 0" />
-            <inertia ixx="0.025" ixy="0" ixz="0" iyy="0.021" iyz="0" izz="0.011" />
+            <inertia ixx="0.0025" ixy="0" ixz="0" iyy="0.0021" iyz="0" izz="0.0011" />
         </inertial>
         <visual>
+            <origin rpy="1.57 0.0 3.14" xyz="0.0 -0.07 0.0" />
             <geometry>
-                <box size=".2 .2 .2" />
+                <mesh filename="package://custom_description/meshes/$(arg robot_type)/payload.STL" scale="1 1 1" />
             </geometry>
         </visual>
@@ -74,5 +75,7 @@
     <xacro:sensor_d435 name="front_camera" topics_ns="$(arg ns)/front_camera" parent="base"
         sim="$(arg sim)">
-        <origin xyz="0.22 0.0 0.05" rpy="0 0.21 0" />
+        <!-- <origin xyz="0.185 0.0 0.115" rpy="0 0.52 0" /> -->
+        <!-- <origin xyz="0.185 0.0 0.235" rpy="0 0.45 0" /> -->
+        <origin xyz="0.185 0.0 0.115" rpy="0 0.45 0" />
     </xacro:sensor_d435>
     <!-- ros_control plugin -->

File: custom_description/urdf/sensor_d435.xacro (robot description, xacro)
@@ -59,5 +59,5 @@
             </inertial>
         </link>
-        <xacro:if value="$(arg sim)">
+        <xacro:if value="${sim}">
             <!-- camera depth joints and links -->
             <joint name="${name}_depth_joint" type="fixed">
