Commit message: add t265 collision

File: custom_description/urdf/sensor_t265.xacro (robot description, xacro)
@@ -39,7 +39,7 @@
             <collision>
                 <origin xyz="0 0 0" rpy="0 0 0"/>
-                <!-- <geometry>
-                    <mesh filename="package://realsense2_description/meshes/t265.stl"/>
-                </geometry> -->
+                <geometry>
+                    <box size="0.01 0.01 0.01" />
+                </geometry>
             </collision>
             <inertial>
